File: kicad/uart_header.kicad_sch (KiCad schematic)
At the start: 3 parts, among them J4 Conn_01x07

Commit message: v1.1
Parts:
- renumbered J4 to J2
Changed lines of the file:
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@@
 		(dnp no)
 		(fields_autoplaced yes)
-		(property "Reference" "J4"
+		(property "Reference" "J2"
 			(at 64.77 29.2099 0)
 			(show_name no)
@@
 			(project "FTDIboard"
 				(path "/aa1b40ca-4f8c-407d-ac45-3b99f0a9bdba/3abb35d5-16d8-4c38-b1b3-cd1430af0acd"
-					(reference "J4")
+					(reference "J2")
 					(unit 1)
 				)
