File: kicad/usb_input.kicad_sch (KiCad schematic)
At the start: 6 parts, among them J1 USB_C_Receptacle_USB2.0_14P, U1 USBLC6-2SC6

Commit message: blenders
Other:
- note removed: "WHAT DO I CONNECT HERE??"
- moved on the sheet: JP1, JP2, U1
Changed lines of the file:
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@@
 	(generator_version "10.0")
 	(paper "A4")
-	(text "WHAT DO I CONNECT HERE??"
-		(exclude_from_sim no)
-		(at 88.9 28.194 0)
-		(effects
-			(font
-				(size 1.27 1.27)
-			)
-		)
-	)
 	(junction
 		(at 31.75 62.23)
@@
 	)
 	(junction
-		(at 69.85 27.94)
+		(at 53.34 38.1)
 		(diameter 0)
 		(color 0 0 0 0)
 	)
 	(junction
-		(at 53.34 38.1)
+		(at 69.85 27.94)
 		(diameter 0)
 		(color 0 0 0 0)
@@
 	(wire
 		(pts
-			(xy 78.74 45.72) (xy 78.74 46.99)
+			(xy 88.9 45.72) (xy 88.9 46.99)
 		)
 		(stroke
@@
 	(wire
 		(pts
-			(xy 114.3 40.64) (xy 116.84 40.64)
+			(xy 124.46 40.64) (xy 127 40.64)
 		)
 		(stroke
@@
 	(wire
 		(pts
-			(xy 83.82 40.64) (xy 104.14 40.64)
+			(xy 93.98 40.64) (xy 114.3 40.64)
 		)
 		(stroke
@@
 	(wire
 		(pts
-			(xy 53.34 40.64) (xy 73.66 40.64)
-		)
-		(stroke
-			(width 0)
-			(type default)
-		)
-	)
-	(wire
-		(pts
-			(xy 78.74 30.48) (xy 78.74 33.02)
+			(xy 53.34 40.64) (xy 83.82 40.64)
+		)
+		(stroke
+			(width 0)
+			(type default)
+		)
+	)
+	(wire
+		(pts
+			(xy 88.9 30.48) (xy 88.9 33.02)
 		)
 		(stroke
@@
 	(wire
 		(pts
-			(xy 114.3 38.1) (xy 116.84 38.1)
-		)
-		(stroke
-			(width 0)
-			(type default)
-		)
-	)
-	(wire
-		(pts
-			(xy 73.66 38.1) (xy 53.34 38.1)
+			(xy 124.46 38.1) (xy 127 38.1)
+		)
+		(stroke
+			(width 0)
+			(type default)
+		)
+	)
+	(wire
+		(pts
+			(xy 83.82 38.1) (xy 53.34 38.1)
 		)
 		(stroke
@@
 	(wire
 		(pts
-			(xy 83.82 38.1) (xy 104.14 38.1)
+			(xy 93.98 38.1) (xy 114.3 38.1)
 		)
 		(stroke
@@
 	(hierarchical_label "USBC_D+"
 		(shape input)
-		(at 116.84 40.64 0)
+		(at 127 40.64 0)
 		(effects
 			(font
@@
 	(hierarchical_label "USBC_D-"
 		(shape input)
-		(at 116.84 38.1 0)
+		(at 127 38.1 0)
 		(effects
 			(font
@@
 	(hierarchical_label "VBUS"
 		(shape input)
-		(at 78.74 30.48 180)
+		(at 88.9 30.48 180)
 		(effects
 			(font
@@
 	(symbol
 		(lib_id "power:GND")
-		(at 78.74 46.99 0)
+		(at 88.9 46.99 0)
 		(unit 1)
 		(body_style 1)
@@
 		(fields_autoplaced yes)
 		(property "Reference" "#PWR03"
-			(at 78.74 53.34 0)
+			(at 88.9 53.34 0)
 			(hide yes)
 			(show_name no)
@@
 		)
 		(property "Value" "GND"
-			(at 78.74 52.07 0)
+			(at 88.9 52.07 0)
 			(show_name no)
 			(do_not_autoplace no)
@@
 		)
 		(property "Footprint" ""
-			(at 78.74 46.99 0)
+			(at 88.9 46.99 0)
 			(hide yes)
 			(show_name no)
@@
 		)
 		(property "Datasheet" ""
-			(at 78.74 46.99 0)
+			(at 88.9 46.99 0)
 			(hide yes)
 			(show_name no)
@@
 		)
 		(property "Description" "Power symbol creates a global label with name \"GND\" , ground"
-			(at 78.74 46.99 0)
+			(at 88.9 46.99 0)
 			(hide yes)
 			(show_name no)
@@
 	(symbol
 		(lib_id "Power_Protection:USBLC6-2SC6")
-		(at 78.74 38.1 0)
+		(at 88.9 38.1 0)
 		(unit 1)
 		(body_style 1)
@@
 		(fields_autoplaced yes)
 		(property "Reference" "U1"
-			(at 80.3911 30.48 0)
+			(at 90.5511 30.48 0)
 			(show_name no)
 			(do_not_autoplace no)
@@
 		)
 		(property "Value" "USBLC6-2SC6"
-			(at 80.3911 33.02 0)
+			(at 90.5511 33.02 0)
 			(show_name no)
 			(do_not_autoplace no)
@@
 		)
 		(property "Footprint" "Package_TO_SOT_SMD:SOT-23-6"
-			(at 80.01 44.45 0)
+			(at 90.17 44.45 0)
 			(hide yes)
 			(show_name no)
@@
 		)
 		(property "Datasheet" "https://www.st.com/resource/en/datasheet/usblc6-2.pdf"
-			(at 80.01 46.355 0)
+			(at 90.17 46.355 0)
 			(hide yes)
 			(show_name no)
@@
 		)
 		(property "Description" "Very low capacitance ESD protection diode, 2 data-line, SOT-23-6"
-			(at 78.74 38.1 0)
+			(at 88.9 38.1 0)
 			(hide yes)
 			(show_name no)
@@
 	(symbol
 		(lib_id "Jumper:SolderJumper_2_Bridged")
-		(at 109.22 40.64 180)
+		(at 119.38 40.64 180)
 		(unit 1)
 		(body_style 1)
@@
 		(dnp no)
 		(property "Reference" "JP2"
-			(at 109.22 46.99 0)
+			(at 119.38 46.99 0)
 			(show_name no)
 			(do_not_autoplace no)
@@
 		)
 		(property "Value" "SolderJumper_2_Bridged"
-			(at 109.22 44.45 0)
+			(at 119.38 44.45 0)
 			(show_name no)
 			(do_not_autoplace no)
@@
 		)
 		(property "Footprint" "Jumper:SolderJumper-2_P1.3mm_Bridged_RoundedPad1.0x1.5mm"
-			(at 109.22 40.64 0)
+			(at 119.38 40.64 0)
 			(hide yes)
 			(show_name no)
@@
 		)
 		(property "Datasheet" ""
-			(at 109.22 34.29 0)
+			(at 119.38 34.29 0)
 			(hide yes)
 			(show_name no)
@@
 		)
 		(property "Description" "Solder Jumper, 2-pole, closed/bridged"
-			(at 109.22 35.56 0)
+			(at 119.38 35.56 0)
 			(hide yes)
 			(show_name no)
@@
 	(symbol
 		(lib_id "Jumper:SolderJumper_2_Bridged")
-		(at 109.22 38.1 0)
+		(at 119.38 38.1 0)
 		(unit 1)
 		(body_style 1)
@@
 		(fields_autoplaced yes)
 		(property "Reference" "JP1"
-			(at 109.22 31.75 0)
+			(at 119.38 31.75 0)
 			(show_name no)
 			(do_not_autoplace no)
@@
 		)
 		(property "Value" "SolderJumper_2_Bridged"
-			(at 109.22 34.29 0)
+			(at 119.38 34.29 0)
 			(show_name no)
 			(do_not_autoplace no)
@@
 		)
 		(property "Footprint" "Jumper:SolderJumper-2_P1.3mm_Bridged_RoundedPad1.0x1.5mm"
-			(at 109.22 38.1 0)
+			(at 119.38 38.1 0)
 			(hide yes)
 			(show_name no)
@@
 		)
 		(property "Datasheet" ""
-			(at 109.22 44.45 0)
+			(at 119.38 44.45 0)
 			(hide yes)
 			(show_name no)
@@
 		)
 		(property "Description" "Solder Jumper, 2-pole, closed/bridged"
-			(at 109.22 43.18 0)
-			(hide yes)
-			(show_name no)
+			(at 119.38 43.18 0)
+			(hide yes)
+			(show_name no)
