File: kicad/FTDIboard.kicad_sch (KiCad schematic)
At the start: 4 parts

Commit message: v1.1
Other:
- sheet USB_UART_CORE ports: added none; removed 5V_USB
Changed lines of the file:
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@@
-	)
-	(junction
-		(at 52.07 68.58)
-		(diameter 0)
-		(color 0 0 0 0)
 	)
 	(junction
@@
 	)
 	(junction
+		(at 54.61 59.69)
+		(diameter 0)
+		(color 0 0 0 0)
+	)
+	(junction
 		(at 119.38 35.56)
 		(diameter 0)
@@
 		(color 0 0 0 0)
 	)
-	(junction
-		(at 54.61 59.69)
-		(diameter 0)
-		(color 0 0 0 0)
-	)
 	(wire
 		(pts
@@
 	(wire
 		(pts
-			(xy 54.61 33.02) (xy 54.61 59.69)
+			(xy 54.61 35.56) (xy 54.61 59.69)
 		)
 		(stroke
@@
 	(wire
 		(pts
-			(xy 52.07 35.56) (xy 52.07 68.58)
-		)
-		(stroke
-			(width 0)
-			(type default)
-		)
-	)
-	(wire
-		(pts
 			(xy 82.55 38.1) (xy 118.11 38.1)
 		)
@@
 	(wire
 		(pts
-			(xy 52.07 35.56) (xy 57.15 35.56)
-		)
-		(stroke
-			(width 0)
-			(type default)
-		)
-	)
-	(wire
-		(pts
 			(xy 115.57 71.12) (xy 124.46 71.12)
 		)
@@
 	(wire
 		(pts
-			(xy 54.61 33.02) (xy 57.15 33.02)
+			(xy 54.61 35.56) (xy 57.15 35.56)
 		)
 		(stroke
@@
 			)
 		)
-		(pin "5V_USB" input
-			(at 57.15 33.02 180)
-			(effects
-				(font
-					(size 1.27 1.27)
-				)
-				(justify left)
-			)
-		)
