File: kicad/led_indicators.kicad_sch (KiCad schematic)
At the start: 40 parts, among them U4 ULN2003, U5 ULN2003

Commit message: v1.1
Parts:
- removed C10, C11: 100nF, Capacitor_SMD:C_0805_2012Metric_Pad1.18x1.45mm_HandSolder, symbol Device:C_Small
- removed C12, C13: 10uF, Capacitor_SMD:C_0805_2012Metric_Pad1.18x1.45mm_HandSolder, symbol Device:C_Small
- removed R19, R20, R21, R22, R23, R24, R26, R27, R28: 10k, Resistor_SMD:R_0805_2012Metric_Pad1.20x1.40mm_HandSolder, symbol Device:R_Small_US
- removed U4, U5: ULN2003, Package_SO:TSSOP-16_4.4x5mm_P0.65mm, symbol Transistor_Array:ULN2003
- added D13: LED, LED_SMD:LED_0805_2012Metric_Pad1.15x1.40mm_HandSolder, symbol Device:LED
- renumbered R9 to R13, R10 to R14, R11 to R15, R12 to R16, R13 to R17, R14 to R18, R15 to R19, R16 to R20, R17 to R21, R18 to R22, R29 to R23, R30 to R24
Connections:
- net GND: now also D13.1 (K)
- net VIO: now also R25.1
- net at D9.2 (A): now also R19.2; no longer R25.2
- net at R13.2: now also D7.2 (A)
- net at R15.2: now also D5.2 (A)
- net at R17.2: now also D3.2 (A)
- net at R20.2: now also D1.2 (A)
- net at D10.2 (A): now also R21.2
- net at D8.2 (A): now also R14.2
- net at R16.2: now also D6.2 (A)
- net at D4.2 (A): now also R18.2
- net at R22.2: now also D2.2 (A)
- new net: D13.2 (A), R25.2
- no-connect marks 8 -> 0
Other:
- moved on the sheet: R13, R14, R15, R16, R17, R18, R19, R20, R21, R22
