File: kicad/power.kicad_sch (KiCad schematic)
At the start: 9 parts, among them Q1 AO3401A, SW1 SW_SPDT_321, U2 TLV75733PDBV

Commit message: v1.1
Parts:
- added F2: 2.5A, Fuse_US_Handsoldering_AKL:Fuse_0603_1608Metric, symbol Device:Polyfuse_Small
Connections:
- net VBUS_PROTECTED: now also F2.2; no longer F1.2
- new net: F1.2, F2.1
Other:
- moved on the sheet: F1
Changed lines of the file:
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@@
 	(text "500-750mA"
 		(exclude_from_sim no)
-		(at 39.624 16.764 0)
+		(at 30.734 16.764 0)
 		(effects
 			(font
@@
 	(wire
 		(pts
-			(xy 41.91 25.4) (xy 45.72 25.4)
+			(xy 33.02 25.4) (xy 45.72 25.4)
 		)
 		(stroke
@@
 	(wire
 		(pts
-			(xy 33.02 25.4) (xy 36.83 25.4)
+			(xy 24.13 25.4) (xy 27.94 25.4)
 		)
 		(stroke
@@
 		(pts
 			(xy 97.79 52.07) (xy 100.33 52.07)
+		)
+		(stroke
+			(width 0)
+			(type default)
+		)
+	)
+	(wire
+		(pts
+			(xy 50.8 25.4) (xy 54.61 25.4)
 		)
 		(stroke
@@
 	(global_label "VBUS_PROTECTED"
 		(shape input)
-		(at 45.72 25.4 0)
+		(at 54.61 25.4 0)
 		(fields_autoplaced yes)
 		(effects
@@
 		)
 		(property "Intersheetrefs" "${INTERSHEET_REFS}"
-			(at 65.2151 25.4 0)
+			(at 74.1051 25.4 0)
 			(hide yes)
 			(show_name no)
@@
 	(hierarchical_label "VBUS_IN"
 		(shape input)
-		(at 33.02 25.4 180)
+		(at 24.13 25.4 180)
 		(effects
 			(font
@@
 	(symbol
 		(lib_id "Device:Polyfuse_Small")
-		(at 39.37 25.4 90)
+		(at 30.48 25.4 90)
 		(unit 1)
 		(body_style 1)
@@
 		(fields_autoplaced yes)
 		(property "Reference" "F1"
-			(at 39.37 19.05 90)
+			(at 30.48 19.05 90)
 			(show_name no)
 			(do_not_autoplace no)
@@
 		)
 		(property "Value" "600mA hold, 1.2A trip"
-			(at 39.37 21.59 90)
+			(at 30.48 21.59 90)
 			(show_name no)
 			(do_not_autoplace no)
@@
 		)
 		(property "Footprint" "Capacitor_THT:C_Disc_D5.1mm_W3.2mm_P5.00mm"
-			(at 44.45 24.13 0)
+			(at 35.56 24.13 0)
 			(hide yes)
 			(show_name no)
@@
 		)
 		(property "Datasheet" ""
-			(at 39.37 25.4 0)
+			(at 30.48 25.4 0)
 			(hide yes)
 			(show_name no)
@@
 		)
 		(property "Description" "Resettable fuse, polymeric positive temperature coefficient, small symbol"
-			(at 39.37 25.4 0)
+			(at 30.48 25.4 0)
 			(hide yes)
 			(show_name no)
@@
 					(unit 1)
 				)
+			)
+		)
+	)
+	(symbol
+		(lib_id "Device:Polyfuse_Small")
+		(at 48.26 25.4 90)
+		(unit 1)
+		(body_style 1)
+		(exclude_from_sim no)
+		(in_bom yes)
+		(on_board yes)
+		(in_pos_files yes)
+		(dnp no)
+		(fields_autoplaced yes)
+		(property "Reference" "F2"
+			(at 48.26 19.05 90)
+			(show_name no)
+			(do_not_autoplace no)
+			(effects
+				(font
+					(size 1.27 1.27)
+				)
+			)
+		)
+		(property "Value" "2.5A"
+			(at 48.26 21.59 90)
+			(show_name no)
+			(do_not_autoplace no)
+			(effects
+				(font
+					(size 1.27 1.27)
+				)
+			)
+		)
+		(property "Footprint" "Fuse_US_Handsoldering_AKL:Fuse_0603_1608Metric"
+			(at 53.34 24.13 0)
+			(hide yes)
+			(show_name no)
+			(do_not_autoplace no)
+			(effects
+				(font
+					(size 1.27 1.27)
+				)
+				(justify left)
+			)
+		)
+		(property "Datasheet" ""
+			(at 48.26 25.4 0)
+			(hide yes)
+			(show_name no)
+			(do_not_autoplace no)
+			(effects
+				(font
+					(size 1.27 1.27)
+				)
+			)
+		)
+		(property "Description" "Resettable fuse, polymeric positive temperature coefficient, small symbol"
+			(at 48.26 25.4 0)
+			(hide yes)
+			(show_name no)
+			(do_not_autoplace no)
+			(effects
+				(font
+					(size 1.27 1.27)
+				)
+			)
+		)
+		(pin "2"
+		)
+		(pin "1"
+		)
+		(instances
+			(project "FTDIboard"
+				(path "/aa1b40ca-4f8c-407d-ac45-3b99f0a9bdba/180d1957-f9a0-47cc-83f3-9f5e477c33e6"
+					(reference "F2")
+					(unit 1)
+				)
