File: kicad/usb_uart_core.kicad_sch (KiCad schematic)
At the start: 9 parts, among them U3 FT232RL

Commit message: arrival
Connections:
- net 5V_USB is gone; now on net VIO: C8.1, C9.1, U3.20 (VCC)
Other:
- note added: "moved from 5vusb"
Changed lines of the file:
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@@
 	(generator_version "10.0")
 	(paper "A4")
+	(text "moved from 5vusb"
+		(exclude_from_sim no)
+		(at 112.268 64.008 0)
+		(effects
+			(font
+				(size 1.27 1.27)
+			)
+		)
+	)
+	(junction
+		(at 104.14 66.04)
+		(diameter 0)
+		(color 0 0 0 0)
+	)
 	(junction
 		(at 88.9 66.04)
@@
 	(junction
 		(at 104.14 127)
-		(diameter 0)
-		(color 0 0 0 0)
-	)
-	(junction
-		(at 104.14 66.04)
 		(diameter 0)
 		(color 0 0 0 0)
@@
 	(wire
 		(pts
+			(xy 99.06 66.04) (xy 104.14 66.04)
+		)
+		(stroke
+			(width 0)
+			(type default)
+		)
+	)
+	(wire
+		(pts
 			(xy 121.92 92.71) (xy 124.46 92.71)
 		)
@@
 	(wire
 		(pts
-			(xy 104.14 62.23) (xy 104.14 66.04)
-		)
-		(stroke
-			(width 0)
-			(type default)
-		)
-	)
-	(wire
-		(pts
 			(xy 121.92 87.63) (xy 124.46 87.63)
 		)
@@
 		(effects
 			(font
-				(size 1.27 1.27)
-			)
-			(justify left)
-		)
-	)
-	(hierarchical_label "5V_USB"
-		(shape input)
-		(at 104.14 62.23 90)
-		(effects
-			(font
